Commit message: Final verified commit for the motoman_mh50_support package

File: motoman_mh50_support/urdf/mh50.urdf (robot description, URDF)
Before this commit: robot motoman_mh50, 8 links, 7 joints
Links:
- added link base
- link base_link: geometry collision mesh filename=package://motoman_mh50_support/meshes/collision/MH50_BASE.s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 scale=0.001 0.001 0.001; visual mesh filename=package://motoman_mh50_support/meshes/visual/MH50_BASE.stl scale=0.001 0.001 0.001
- link link_b: geometry collision mesh filename=package://motoman_mh50_support/meshes/collision/MH50_B_AXIS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 scale=0.001 0.001 0.001; visual mesh filename=package://motoman_mh50_support/meshes/visual/MH50_B_AXIS.stl scale=0.001 0.001 0.001
- link link_l: geometry collision mesh filename=package://motoman_mh50_support/meshes/collision/MH50_L_AXIS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 scale=0.001 0.001 0.001; visual mesh filename=package://motoman_mh50_support/meshes/visual/MH50_L_AXIS.stl scale=0.001 0.001 0.001
- link link_r: geometry collision mesh filename=package://motoman_mh50_support/meshes/collision/MH50_R_AXIS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 scale=0.001 0.001 0.001; visual mesh filename=package://motoman_mh50_support/meshes/visual/MH50_R_AXIS.stl scale=0.001 0.001 0.001
- link link_s: geometry collision mesh filename=package://motoman_mh50_support/meshes/collision/MH50_S_AXIS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 scale=0.001 0.001 0.001; visual mesh filename=package://motoman_mh50_support/meshes/visual/MH50_S_AXIS.stl scale=0.001 0.001 0.001
- link link_t: geometry collision mesh filename=package://motoman_mh50_support/meshes/collision/MH50_T_AXIS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 scale=0.001 0.001 0.001; visual mesh filename=package://motoman_mh50_support/meshes/visual/MH50_T_AXIS.stl scale=0.001 0.001 0.001
- link link_u: geometry collision mesh filename=package://motoman_mh50_support/meshes/collision/MH50_U_AXIS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 scale=0.001 0.001 0.001; visual mesh filename=package://motoman_mh50_support/meshes/visual/MH50_U_AXIS.stl scale=0.001 0.001 0.001
Joints:
- removed joint link_6-tool0
- added joint base_link-base: type fixed, parent base_link, child base, origin xyz=0 0 0.540 rpy=0 0 0
- added joint joint_t-tool0: type fixed, parent link_t, child tool0, origin xyz=0.175 0 0 rpy=3.1415926 -1.570796 0
- joint joint_b: limit lower=-2.1817 upper=2.1817 effort=100 velocity=3.48 -> lower=-2.18167 upper=2.18167 effort=706.08 velocity=4.363; origin xyz=0.7065 0 0 rpy=0 0 0 -> xyz=0 0 0 rpy=0 0 0
- joint joint_l: limit lower=-1.5708 upper=2.35619 effort=100 velocity=2.96 -> lower=-1.57079 upper=2.35619 effort=6276.26 velocity=3.103; origin xyz=0.145 -0.1455 0.281 rpy=0 0 0 -> xyz=0.145 0 0 rpy=0 0 0
- joint joint_r: limit lower=-6.28319 upper=6.28319 effort=100 velocity=3.48 -> lower=-6.28319 upper=6.28319 effort=823.76 velocity=4.363; origin xyz=0.306 0.155 0.210 rpy=0 0 0 -> xyz=1.025 0 0.210 rpy=0 0 0
- joint joint_s: limit lower=-3.14159 upper=3.14159 effort=100 velocity=2.96 -> lower=-3.14159 upper=3.14159 effort=4903.32 velocity=3.141; origin xyz=0 0 0.259 rpy=0 0 0 -> xyz=0 0 0.540 rpy=0 0 0
- joint joint_t: limit lower=-6.2831 upper=6.2831 effort=100 velocity=6.97 -> lower=-6.2831 upper=6.2831 effort=333.43 velocity=6.283; origin xyz=0.1595 0 0 rpy=0 0 0 -> xyz=0 0 0 rpy=0 0 0
- joint joint_u: limit lower=-1.55 upper=4.014 effort=100 velocity=2.96 -> lower=-1.39626 upper=3.59538 effort=2745.86 velocity=3.106; origin xyz=-0.0 -0.0095 0.870 rpy=0 0 0 -> xyz=0 0 0.870 rpy=0 0 0

File: motoman_mh50_support/urdf/mh50_macro.xacro (robot description, xacro)
@@ -1,163 +1,173 @@
 <?xml version="1.0" ?>
 <robot xmlns:xacro="http://ros.org/wiki/xacro">
-	<property name="pi" value="3.14157"/>
-	<xacro:macro name="motoman_mh50" params="prefix">
-		<!-- link list -->
-		<link name="${prefix}base_link">
-			<visual>
-			        <origin rpy="0 0 0"/>
-				<geometry>
-					<mesh filename="package://motoman_mh50_support/meshes/mh50/visual/MH50_BASE_AXIS.dae" />
-				</geometry>
-				<material name="blue">
-					<color rgba="0.8 0.8 .8 1"/>
-				</material>
-			</visual>
-			<collision>
-			        <origin rpy="0 0 0" xyz="-0.086 0 0.1295"/>
-				<geometry>
-					<box size="0.635 0.470 0.259"/>
-				</geometry>
-			</collision>
-		</link>
-		<link name="${prefix}link_s">
-			<visual>
-				<geometry>
-					<mesh filename="package://motoman_mh50_support/meshes/mh50/visual/MH50_S_AXIS.dae"/>
-				</geometry>
-			</visual>
-			<collision>
-				<geometry>
-					<mesh filename="package://motoman_mh50_support/meshes/mh50/collision/MH50_S_AXIS.dae" />
-				</geometry>
-			</collision>
-		</link>
-		<link name="${prefix}link_l">
-			<visual>
-				<!-- <origin rpy="1.57 3.1416 0" xyz="0 0 0"/> -->
-				<geometry>
-					<mesh filename="package://motoman_mh50_support/meshes/mh50/visual/MH50_L_AXIS.dae"/>
-				</geometry>
-			</visual>
-			<collision>
-				<!-- <origin rpy="1.57 3.1416 0" xyz="0 0 0"/> -->
-				<geometry>
-					<mesh filename="package://motoman_mh50_support/meshes/mh50/collision/MH50_L_AXIS.dae" />
-				</geometry>
-			</collision>
-		</link>
-		<link name="${prefix}link_u">
-			<visual>
-				<!-- <origin rpy="1.57 -3.1415 0" xyz="0 0 0"/> -->
-				<geometry>
-					<mesh filename="package://motoman_mh50_support/meshes/mh50/visual/MH50_U_AXIS.dae"/>
-				</geometry>
-			</visual>
-			<collision>
-				<!-- <origin rpy="1.57 -3.1415 0" xyz="0 0 0"/> -->
-				<geometry>
-					<mesh filename="package://motoman_mh50_support/meshes/mh50/collision/MH50_U_AXIS.dae" />
-				</geometry>
-			</collision>
-		</link>
-		<link name="${prefix}link_r">
-			<visual>
-				<!-- <origin rpy="0 0 3.1416" xyz="0 0 0"/> -->
-				<geometry>
-					<mesh filename="package://motoman_mh50_support/meshes/mh50/visual/MH50_R_AXIS.dae"/>
-				</geometry>
-			</visual>
-			<collision>
-				<!-- <origin rpy="0 0 3.1416" xyz="0 0 0"/> -->
-				<geometry>
-					<mesh filename="package://motoman_mh50_support/meshes/mh50/collision/MH50_R_AXIS.dae" />
-				</geometry>
-			</collision>
-		</link>
-		<link name="${prefix}link_b">
-			<visual>
-				<!-- <origin rpy="-1.57 0 3.1416" xyz="0 0 0"/> -->
-				<geometry>
-					<mesh filename="package://motoman_mh50_support/meshes/mh50/visual/MH50_B_AXIS.dae"/>
-				</geometry>
-				<material name="blue"/>
-			</visual>
-			<collision>
-				<!-- <origin rpy="-1.57 0 3.1416" xyz="0 0 0"/> -->
-				<geometry>
-					<mesh filename="package://motoman_mh50_support/meshes/mh50/collision/MH50_B_AXIS.dae" />
-				</geometry>
-			</collision>
-		</link>
-		<link name="${prefix}link_t">
-			<visual>
-				<geometry>
-					<mesh filename="package://motoman_mh50_support/meshes/mh50/visual/MH50_T_AXIS.dae" />
-				</geometry>
-			</visual>
-			<collision>
-				<geometry>
-					<mesh filename="package://motoman_mh50_support/meshes/mh50/collision/MH50_T_AXIS.dae" />
-				</geometry>
-				<material name="yellow"/>
-			</collision>
-		</link>
-		<!-- end of link list -->
-		<!-- joint list -->
-		<joint name="${prefix}joint_s" type="revolute">
-			<parent link="${prefix}base_link"/>
-			<child link="${prefix}link_s"/>
-			<origin xyz="0 0 0.259" rpy="0 0 0"/>
-			<axis xyz="0 0 1" />
-			<limit lower="-3.14159" upper="3.14159" effort="100" velocity="2.96" />
-		</joint>
-		<joint name="${prefix}joint_l" type="revolute">
-			<parent link="${prefix}link_s"/>
-			<child link="${prefix}link_l"/>
-			<origin xyz="0.145 -0.1455 0.281" rpy="0 0 0"/>
-			<axis xyz="0 1 0" />
-			<limit lower="-1.5708" upper="2.35619" effort="100" velocity="2.96" />
-		</joint>
-		<joint name="${prefix}joint_u" type="revolute">
-			<parent link="${prefix}link_l"/>
-			<child link="${prefix}link_u"/>
-			<origin xyz="-0.0 -0.0095 0.870" rpy="0 0 0"/>
-			<axis xyz="0 -1 0" />
-	      <!-- Old limits: lower="-2.96706" upper="4.38078"
-                   The new limits below were measured from an MH50F.  They ensure
- 		   that link_r won't hit link_l even when joint_r is at 45 degrees.
-		   The old limits were converted directly from the MH50 data sheet,
-		   which was clearly way off. -->
-			<limit lower="-1.55" upper="4.014" effort="100" velocity="2.96" />
-		</joint>
-		<joint name="${prefix}joint_r" type="revolute">
-			<parent link="${prefix}link_u"/>
-			<child link="${prefix}link_r"/>
-			<origin xyz="0.306 0.155 0.210" rpy="0 0 0"/>
-			<axis xyz="-1 0 0" />
-			<limit lower="-6.28319" upper="6.28319" effort="100" velocity="3.48" />
-		</joint>
-		<joint name="${prefix}joint_b" type="revolute">
-			<parent link="${prefix}link_r"/>
-			<child link="${prefix}link_b"/>
-			<origin xyz="0.7065 0 0" rpy="0 0 0"/>
-			<axis xyz="0 -1 0" />
-			<limit lower="-2.1817" upper="2.1817" effort="100" velocity="3.48" />
-		</joint>
-		<joint name="${prefix}joint_t" type="revolute">
-			<parent link="${prefix}link_b"/>
-			<child link="${prefix}link_t"/>
-			<origin xyz="0.1595 0 0" rpy="0 0 0"/>
-			<axis xyz="-1 0 0" />
-			<limit lower="-6.2831" upper="6.2831" effort="100" velocity="6.97" />
-		</joint>
-		<!-- end of joint list -->
-	   	<!-- ROS-Industrial 'tool0' frame: all-zeros tool frame -->
-	    	<link name="${prefix}tool0" />
-	    	<joint name="${prefix}link_6-tool0" type="fixed">
-	      		<origin xyz="0.0155 0 0" rpy="${pi} ${-pi/2.0} 0" />
-	      		<parent link="${prefix}link_t" />
-	      		<child link="${prefix}tool0" />
-	    	</joint>
-	</xacro:macro>
+<xacro:macro name="motoman_mh50" params="prefix">
+    <!-- Properties -->
+    <material name="yaskawa_blue">
+          <color rgba="0.12941 0.14902 0.74902 1" />
+    </material>
+    <!-- link list -->
+    <link name="${prefix}base_link">
+        <visual>
+            <origin xyz="0 0 0" rpy="0 0 0" />
+            <geometry>
+                <mesh filename="package://motoman_mh50_support/meshes/visual/MH50_BASE.stl" scale="0.001 0.001 0.001"/>
+            </geometry>
+            <material name="yaskawa_blue"/>
+        </visual>
+        <collision>
+            <origin xyz="0 0 0" rpy="0 0 0" />
+            <geometry>
+                <mesh filename="package://motoman_mh50_support/meshes/collision/MH50_BASE.stl" scale="0.001 0.001 0.001"/>
+            </geometry>
+        </collision>
+    </link>
+    <link name="${prefix}link_s">
+        <visual>
+            <origin xyz="0 0 -0.540" rpy="0 0 0" />
+            <geometry>
+                <mesh filename="package://motoman_mh50_support/meshes/visual/MH50_S_AXIS.stl" scale="0.001 0.001 0.001"/>
+            </geometry>
+            <material name="yaskawa_blue"/>
+        </visual>
+        <collision>
+            <origin xyz="0 0 -0.540" rpy="0 0 0" />
+            <geometry>
+                <mesh filename="package://motoman_mh50_support/meshes/collision/MH50_S_AXIS.stl" scale="0.001 0.001 0.001"/>
+            </geometry>
+        </collision>
+    </link>
+    <link name="${prefix}link_l">
+        <visual>
+            <origin xyz="-0.145 0 -0.540" rpy="0 0 0" />
+            <geometry>
+                <mesh filename="package://motoman_mh50_support/meshes/visual/MH50_L_AXIS.stl" scale="0.001 0.001 0.001"/>
+            </geometry>
+            <material name="yaskawa_blue"/>
+        </visual>
+        <collision>
+            <origin xyz="-0.145 0 -0.540" rpy="0 0 0" />
+            <geometry>
+                <mesh filename="package://motoman_mh50_support/meshes/collision/MH50_L_AXIS.stl" scale="0.001 0.001 0.001"/>
+            </geometry>
+        </collision>
+    </link>
+    <link name="${prefix}link_u">
+        <visual>
+            <origin xyz="-0.145 0 -1.410" rpy="0 0 0" />
+            <geometry>
+                <mesh filename="package://motoman_mh50_support/meshes/visual/MH50_U_AXIS.stl" scale="0.001 0.001 0.001"/>
+            </geometry>
+            <material name="yaskawa_blue"/>
+        </visual>
+        <collision>
+            <origin xyz="-0.145 0 -1.410" rpy="0 0 0" />
+            <geometry>
+                <mesh filename="package://motoman_mh50_support/meshes/collision/MH50_U_AXIS.stl" scale="0.001 0.001 0.001"/>
+            </geometry>
+        </collision>
+    </link>
+    <link name="${prefix}link_r">
+        <visual>
+            <origin xyz="-1.170 0 -1.620" rpy="0 0 0" />
+            <geometry>
+                <mesh filename="package://motoman_mh50_support/meshes/visual/MH50_R_AXIS.stl" scale="0.001 0.001 0.001"/>
+            </geometry>
+            <material name="yaskawa_blue"/>
+        </visual>
+        <collision>
+            <origin xyz="-1.170 0 -1.620" rpy="0 0 0" />
+            <geometry>
+                <mesh filename="package://motoman_mh50_support/meshes/collision/MH50_R_AXIS.stl" scale="0.001 0.001 0.001"/>
+            </geometry>
+        </collision>
+    </link>
+    <link name="${prefix}link_b">
+        <visual>
+            <origin xyz="-1.170 0 -1.620" rpy="0 0 0" />
+            <geometry>
+                <mesh filename="package://motoman_mh50_support/meshes/visual/MH50_B_AXIS.stl" scale="0.001 0.001 0.001"/>
+            </geometry>
+            <material name="yaskawa_blue"/>
+        </visual>
+        <collision>
+            <origin xyz="-1.170 0 -1.620" rpy="0 0 0"/>
+            <geometry>
+                <mesh filename="package://motoman_mh50_support/meshes/collision/MH50_B_AXIS.stl" scale="0.001 0.001 0.001"/>
+            </geometry>
+        </collision>
+    </link>
+    <link name="${prefix}link_t">
+        <visual>
+            <origin xyz="-1.170 0 -1.620" rpy="0 0 0" />
+            <geometry>
+                <mesh filename="package://motoman_mh50_support/meshes/visual/MH50_T_AXIS.stl" scale="0.001 0.001 0.001"/>
+            </geometry>
+            <material name="yaskawa_blue"/>
+        </visual>
+        <collision>
+            <origin xyz="-1.170 0 -1.620" rpy="0 0 0" />
+            <geometry>
+                <mesh filename="package://motoman_mh50_support/meshes/collision/MH50_T_AXIS.stl" scale="0.001 0.001 0.001"/>
+            </geometry>
+        </collision>
+    </link>
+    <link name="${prefix}tool0"/>
+    <!-- end of link list -->
+    <!-- joint list -->
+    <joint name="${prefix}joint_s" type="revolute">
+        <parent link="${prefix}base_link"/>
+        <child link="${prefix}link_s"/>
+        <origin xyz="0 0 0.540" rpy="0 0 0" />
+        <axis xyz="0 0 1" />
+        <limit lower="-3.14159" upper="3.14159" effort="4903.32" velocity="3.141"/>
+    </joint>
+    <joint name="${prefix}joint_l" type="revolute">
+        <parent link="${prefix}link_s"/>
+        <child link="${prefix}link_l"/>
+        <origin xyz="0.145 0 0" rpy="0 0 0" />
+        <axis xyz="0 1 0" />
+        <limit lower="-1.57079" upper="2.35619" effort="6276.26" velocity="3.103"/>
+    </joint>
+    <joint name="${prefix}joint_u" type="revolute">
+        <parent link="${prefix}link_l"/>
+        <child link="${prefix}link_u"/>
+        <origin xyz="0 0 0.870" rpy="0 0 0" />
+        <axis xyz="0 -1 0" />
+        <limit lower="-1.39626" upper="3.59538" effort="2745.86" velocity="3.106"/>
+    </joint>
+    <joint name="${prefix}joint_r" type="revolute">
+        <parent link="${prefix}link_u"/>
+        <child link="${prefix}link_r"/>
+        <origin xyz="1.025 0 0.210" rpy="0 0 0"/>
+        <axis xyz="-1 0 0" />
+        <limit lower="-6.28319" upper="6.28319" effort="823.76" velocity="4.363"/>
+    </joint>
+    <joint name="${prefix}joint_b" type="revolute">
+        <parent link="${prefix}link_r"/>
+        <child link="${prefix}link_b"/>
+        <origin xyz="0 0 0" rpy="0 0 0" />
+        <axis xyz="0 -1 0" />
+        <limit lower="-2.18167" upper="2.18167" effort="706.08" velocity="4.363"/>
+    </joint>
+    <joint name="${prefix}joint_t" type="revolute">
+        <parent link="${prefix}link_b"/>
+        <child link="${prefix}link_t"/>
+        <origin xyz="0 0 0" rpy="0 0 0" />
+        <axis xyz="-1 0 0" />
+        <limit lower="-6.2831" upper="6.2831" effort="333.43" velocity="6.283"/>
+    </joint>
+    <joint name="${prefix}joint_t-tool0" type="fixed">
+        <origin xyz="0.175 0 0" rpy="3.1415926 -1.570796 0"/>
+        <parent link="${prefix}link_t"/>
+        <child link="${prefix}tool0"/>
+    </joint>
+    <!-- end of joint list -->
+    <!-- ROS base_link to Robot Manufacturer World Coordinates transform -->
+    <link name="${prefix}base" />
+    <joint name="${prefix}base_link-base" type="fixed">
+        <origin xyz="0 0 0.540" rpy="0 0 0"/>
+        <parent link="${prefix}base_link"/>
+        <child link="${prefix}base"/>
+    </joint>
+    </xacro:macro>
 </robot>
